File: hardware/pi-relay-board-smd/pi-relay-board-smd.kicad_sch (KiCad schematic)
At the start: 1 part, among them J1 Raspberry_Pi_2_3

Commit message: fix: final finishes
Parts:
- J1: footprint Connector_PinHeader_2.54mm:PinHeader_2x20_P2.54mm_Vertical -> Connector_PinHeader_2.54mm:PinHeader_2x20_P2.54mm_Vertical_SMD
Connections:
- net Relay Pin 3/K is gone; now on net Relay Pin 9/K: J1.37 (GPIO26)
- net Relay Pin 10/K: now also J1.13 (GPIO27); no longer J1.15 (GPIO22)
- net Relay Pin 4/K: now also J1.11 (GPIO17); no longer J1.36 (GPIO16)
- net Relay Pin 5/K: now also J1.15 (GPIO22); no longer J1.22 (GPIO25)
- net Relay Pin 6/K: now also J1.16 (GPIO23); no longer J1.18 (GPIO24)
- net Relay Pin 7/K: now also J1.18 (GPIO24); no longer J1.16 (GPIO23)
- net Relay Pin 8/K: now also J1.22 (GPIO25); no longer J1.11 (GPIO17)
- net Relay Pin 9/K: no longer J1.13 (GPIO27)
- new net GPIO16: J1.36 (GPIO16)
