File: hardware/pi-relay-board-smd/relay_pin.kicad_sch (KiCad schematic)
At the start: 4 parts, among them J18 Conn_01x02_Socket, K2 TIANBO-HJR-4102-L, Q1 BC547

Commit message: fix: final finishes
Parts:
- removed J18: Conn_01x02_Socket, TerminalBlock_Phoenix:TerminalBlock_Phoenix_MKDS-1,5-2-5.08_1x02_P5.08mm_Horizontal, symbol Connector:Conn_01x02_Socket
- added J3: Conn_01x03_Socket, TerminalBlock_Phoenix:TerminalBlock_Phoenix_PT-1,5-3-3.5-H_1x03_P3.50mm_Horizontal, symbol Connector:Conn_01x03_Socket
- Q1: footprint Package_TO_SOT_THT:TO-92L_Inline_Wide -> Package_TO_SOT_SMD:SOT-23
- R2: footprint Resistor_THT:R_Axial_DIN0207_L6.3mm_D2.5mm_P7.62mm_Horizontal -> Resistor_SMD:R_0805_2012Metric_Pad1.20x1.40mm_HandSolder
Connections:
- net at K2.1: now also J3.2 (Pin_2)
- net at K2.6: now also J3.1 (Pin_1)
- net at K2.7: now also J3.3 (Pin_3)
Changed lines of the file:
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@@
 	(wire
 		(pts
-			(xy 139.7 91.44) (xy 139.7 88.9)
+			(xy 137.16 83.82) (xy 139.7 83.82)
 		)
 		(stroke
@@
 	(wire
 		(pts
-			(xy 139.7 91.44) (xy 120.65 91.44)
+			(xy 137.16 90.17) (xy 137.16 83.82)
 		)
 		(stroke
@@
 	(wire
 		(pts
+			(xy 135.89 81.28) (xy 139.7 81.28)
+		)
+		(stroke
+			(width 0)
+			(type default)
+		)
+	)
+	(wire
+		(pts
+			(xy 120.65 90.17) (xy 137.16 90.17)
+		)
+		(stroke
+			(width 0)
+			(type default)
+		)
+	)
+	(wire
+		(pts
 			(xy 96.52 68.58) (xy 95.25 68.58)
 		)
@@
 	(wire
 		(pts
-			(xy 120.65 83.82) (xy 120.65 91.44)
+			(xy 120.65 83.82) (xy 120.65 90.17)
 		)
 		(stroke
@@
 			)
 		)
-		(property "Footprint" "Package_TO_SOT_THT:TO-92L_Inline_Wide"
+		(property "Footprint" "Package_TO_SOT_SMD:SOT-23"
 			(at 115.57 70.485 0)
 			(effects
@@
 		)
 		(instances
-			(project "pi-relay-board"
+			(project "pi-relay-board-smd"
 				(path "/d2fef91f-5840-4773-b01e-415a95bac3ff/691f66ce-a9a7-4210-8330-e484efbc945d"
 					(reference "Q1")
@@
 		)
 		(instances
-			(project "pi-relay-board"
+			(project "pi-relay-board-smd"
 				(path "/d2fef91f-5840-4773-b01e-415a95bac3ff/691f66ce-a9a7-4210-8330-e484efbc945d"
 					(reference "#PWR02")
@@
 			)
 		)
-		(property "Footprint" "Resistor_THT:R_Axial_DIN0207_L6.3mm_D2.5mm_P7.62mm_Horizontal"
+		(property "Footprint" "Resistor_SMD:R_0805_2012Metric_Pad1.20x1.40mm_HandSolder"
 			(at 100.33 70.358 90)
 			(effects
@@
 		)
 		(instances
-			(project "pi-relay-board"
+			(project "pi-relay-board-smd"
 				(path "/d2fef91f-5840-4773-b01e-415a95bac3ff/691f66ce-a9a7-4210-8330-e484efbc945d"
 					(reference "R2")
@@
 		)
 		(instances
-			(project "pi-relay-board"
+			(project "pi-relay-board-smd"
 				(path "/d2fef91f-5840-4773-b01e-415a95bac3ff/691f66ce-a9a7-4210-8330-e484efbc945d"
 					(reference "K2")
@@
 				(path "/d2fef91f-5840-4773-b01e-415a95bac3ff/e35df33e-9fd4-4492-8686-e97c7371f93f"
 					(reference "K10")
+					(unit 1)
+				)
+			)
+		)
+	)
+	(symbol
+		(lib_id "Connector:Conn_01x03_Socket")
+		(at 144.78 83.82 0)
+		(mirror x)
+		(unit 1)
+		(exclude_from_sim no)
+		(in_bom yes)
+		(on_board yes)
+		(dnp no)
+		(property "Reference" "J3"
+			(at 146.05 85.0901 0)
+			(effects
+				(font
+					(size 1.27 1.27)
+				)
+				(justify left)
+			)
+		)
+		(property "Value" "Conn_01x03_Socket"
+			(at 146.05 82.5501 0)
+			(effects
+				(font
+					(size 1.27 1.27)
+				)
+				(justify left)
+			)
+		)
+		(property "Footprint" "TerminalBlock_Phoenix:TerminalBlock_Phoenix_PT-1,5-3-3.5-H_1x03_P3.50mm_Horizontal"
+			(at 144.78 83.82 0)
+			(effects
+				(font
+					(size 1.27 1.27)
+				)
+				(hide yes)
+			)
+		)
+		(property "Datasheet" "~"
+			(at 144.78 83.82 0)
+			(effects
+				(font
+					(size 1.27 1.27)
+				)
+				(hide yes)
+			)
+		)
+		(property "Description" "Generic connector, single row, 01x03, script generated"
+			(at 144.78 83.82 0)
+			(effects
+				(font
+					(size 1.27 1.27)
+				)
+				(hide yes)
+			)
+		)
+		(pin "1"
+		)
+		(pin "2"
+		)
+		(pin "3"
+		)
+		(instances
+			(project "pi-relay-board-smd"
+				(path "/d2fef91f-5840-4773-b01e-415a95bac3ff/691f66ce-a9a7-4210-8330-e484efbc945d"
+					(reference "J3")
+					(unit 1)
+				)
+				(path "/d2fef91f-5840-4773-b01e-415a95bac3ff/e003dbba-e903-4928-939e-ed45384c32ae"
+					(reference "J2")
+					(unit 1)
+				)
+				(path "/d2fef91f-5840-4773-b01e-415a95bac3ff/4104c2a8-b10b-4814-8630-4176455720ff"
+					(reference "J4")
+					(unit 1)
+				)
+				(path "/d2fef91f-5840-4773-b01e-415a95bac3ff/4160e499-e228-48ff-bf19-fbbc4f79d536"
+					(reference "J5")
+					(unit 1)
+				)
+				(path "/d2fef91f-5840-4773-b01e-415a95bac3ff/57158c3d-53e9-4aea-9df5-f221bf193187"
+					(reference "J6")
+					(unit 1)
+				)
+				(path "/d2fef91f-5840-4773-b01e-415a95bac3ff/1516f555-b572-405c-8e26-5409c4128995"
+					(reference "J7")
+					(unit 1)
+				)
+				(path "/d2fef91f-5840-4773-b01e-415a95bac3ff/118fbb03-b0f5-4e81-9827-73e518015949"
+					(reference "J8")
+					(unit 1)
+				)
+				(path "/d2fef91f-5840-4773-b01e-415a95bac3ff/a3c9cc38-888b-4558-9948-ff007dba1d89"
+					(reference "J9")
+					(unit 1)
+				)
+				(path "/d2fef91f-5840-4773-b01e-415a95bac3ff/85065515-af0d-46e8-9ec7-79bcf82b83a9"
+					(reference "J10")
+					(unit 1)
+				)
+				(path "/d2fef91f-5840-4773-b01e-415a95bac3ff/e35df33e-9fd4-4492-8686-e97c7371f93f"
+					(reference "J11")
 					(unit 1)
 				)
@@
 		)
 		(instances
-			(project "pi-relay-board"
+			(project "pi-relay-board-smd"
 				(path "/d2fef91f-5840-4773-b01e-415a95bac3ff/1516f555-b572-405c-8e26-5409c4128995"
 					(reference "#PWR019")
@@
 					(unit 1)
 				)
-			)
-		)
-	)
-	(symbol
-		(lib_id "Connector:Conn_01x02_Socket")
-		(at 144.78 86.36 0)
-		(unit 1)
-		(exclude_from_sim no)
-		(in_bom yes)
-		(on_board yes)
-		(dnp no)
-		(fields_autoplaced yes)
-		(property "Reference" "J18"
-			(at 146.05 86.3599 0)
-			(effects
-				(font
-					(size 1.27 1.27)
-				)
-				(justify left)
-			)
-		)
-		(property "Value" "Conn_01x02_Socket"
-			(at 146.05 88.8999 0)
-			(effects
-				(font
-					(size 1.27 1.27)
-				)
-				(justify left)
-			)
-		)
-		(property "Footprint" "TerminalBlock_Phoenix:TerminalBlock_Phoenix_MKDS-1,5-2-5.08_1x02_P5.08mm_Horizontal"
-			(at 144.78 86.36 0)
-			(effects
-				(font
-					(size 1.27 1.27)
-				)
-				(hide yes)
-			)
-		)
-		(property "Datasheet" "~"
-			(at 144.78 86.36 0)
-			(effects
-				(font
-					(size 1.27 1.27)
-				)
-				(hide yes)
-			)
-		)
-		(property "Description" "Generic connector, single row, 01x02, script generated"
-			(at 144.78 86.36 0)
-			(effects
-				(font
-					(size 1.27 1.27)
-				)
-				(hide yes)
-			)
-		)
-		(pin "2"
-		)
-		(pin "1"
-		)
-		(instances
-			(project "pi-relay-board"
-				(path "/d2fef91f-5840-4773-b01e-415a95bac3ff/118fbb03-b0f5-4e81-9827-73e518015949"
-					(reference "J18")
-					(unit 1)
-				)
-				(path "/d2fef91f-5840-4773-b01e-415a95bac3ff/691f66ce-a9a7-4210-8330-e484efbc945d"
-					(reference "J12")
-					(unit 1)
-				)
-				(path "/d2fef91f-5840-4773-b01e-415a95bac3ff/e003dbba-e903-4928-939e-ed45384c32ae"
-					(reference "J13")
-					(unit 1)
-				)
-				(path "/d2fef91f-5840-4773-b01e-415a95bac3ff/4104c2a8-b10b-4814-8630-4176455720ff"
-					(reference "J14")
-					(unit 1)
-				)
-				(path "/d2fef91f-5840-4773-b01e-415a95bac3ff/4160e499-e228-48ff-bf19-fbbc4f79d536"
-					(reference "J15")
-					(unit 1)
-				)
-				(path "/d2fef91f-5840-4773-b01e-415a95bac3ff/57158c3d-53e9-4aea-9df5-f221bf193187"
-					(reference "J16")
-					(unit 1)
-				)
-				(path "/d2fef91f-5840-4773-b01e-415a95bac3ff/1516f555-b572-405c-8e26-5409c4128995"
-					(reference "J17")
-					(unit 1)
-				)
-				(path "/d2fef91f-5840-4773-b01e-415a95bac3ff/a3c9cc38-888b-4558-9948-ff007dba1d89"
-					(reference "J19")
-					(unit 1)
-				)
-				(path "/d2fef91f-5840-4773-b01e-415a95bac3ff/85065515-af0d-46e8-9ec7-79bcf82b83a9"
-					(reference "J20")
-					(unit 1)
-				)
-				(path "/d2fef91f-5840-4773-b01e-415a95bac3ff/e35df33e-9fd4-4492-8686-e97c7371f93f"
-					(reference "J21")
-					(unit 1)
-				)
